File: ww101-shield/eagle/ww101board.sch (EAGLE design)
At the start: 6 parts, among them U1 LIGHTSENSORALS

Commit message: Power routing done... now try signal routing
Parts:
- removed U$1: ARDUINO_R3_SHIELD, SparkFun-Boards:ARDUINO_R3_SHIELD
- added ALS: ALS, IOTExpert:ALS
- added B0, B1, B2, B3: (no value), PatternAgents-TouchWidgets:BUTTON_PASSIVE10MM
- added C1, C3, C5, C8: 1uF, PatternAgents-ProtoPads:CAP0603-CAP
- added C10, C2, C4, C6, C7, C9: 0.1uF, PatternAgents-ProtoPads:CAP0603-CAP
- added C11: 180pF, PatternAgents-ProtoPads:CAP0603-CAP
- added C12, C13, C14: (no value), PatternAgents-ProtoPads:CAP0603-CAP
- added JMP1: (no value), PatternAgents-ProtoPads:JMP-3-NO-PTH
- added JMP2: (no value), PatternAgents-ProtoPads:JMP-3-NO-0603
- added JP1: (no value), SparkFun-Connectors:M05LOCK
- added MB0, MB1: EVQPE1, IOTExpert:EVQPE1
- added MBLED0, MBLED1, ULED0, ULED1, ULED2, ULED3: (no value), adafruit:LEDCHIP-LED0603
- added R10, R9: 10K, PatternAgents-ProtoPads:RESISTOR0603
- added R11: THERMISTOR-5, varistor:THERMISTOR-5
- added R12: 220K, PatternAgents-ProtoPads:RESISTOR0603
- added R13, R14, R15, R16: 560, PatternAgents-ProtoPads:RESISTOR0603
- added R17: 0, PatternAgents-ProtoPads:RESISTOR0603
- added R2: (no value), pot:TRIM_US-3386P
- added R3, R4, R5, R6, R7, R8: 330, PatternAgents-ProtoPads:RESISTOR0603
- added U$5: JMP-3-2_3, PatternAgents-ProtoPads:JMP-3-2_3
- added U$7: CY8C4A45-48, PatternAgents-Cypress:CY8C4A45-48
- R1: value THERMISTOR-5 -> (none); device varistor:THERMISTOR-5 -> PatternAgents-ProtoPads:RESISTOR0603
- U$3: value CY8C4247AZI-L433 -> HPP801A031; device PatternAgents-Cypress:CY8C4247AZI-L433 -> IOTExpert:HPP801A031
- U$4: value HPP801A031 -> JMP-3-1_2; device IOTExpert:HPP801A031 -> PatternAgents-ProtoPads:JMP-3-1_2
- U1: value LIGHTSENSORALS -> ARDUINO_SHIELDNOHOLESORLABELS; device SparkFun-Sensors:LIGHTSENSORALS -> SparkFun-Boards:ARDUINO_SHIELDNOHOLESORLABELS
Connections:
- new net A0: R17.1, U1.A0
- new net CAP-PROX: U$7.P2[5]
- new net CB0: R13.1, U$7.P5[0]
- new net CB1: R14.1, U$7.P5[1]
- new net CB2: R15.1, U$7.P1[7]
- new net CB3: R16.1, U$7.P1[4]
- new net CBLED0: R3.1, U$7.P1[6]
- new net CBLED1: R4.1, U$7.P1[5]
- new net CBLED2: R5.1, U$7.P2[0]
- new net CBLED3: R6.1, U$7.P2[6]
- new net CMOD: C12.1, U$7.P5[2]
- new net CSHIELD: U$7.P3[3]
- new net CTANK: C14.1, U$7.P5[3]
- new net D10: U$7.P0[7], U1.*D10
- new net D3: U$7.P0[3], U1.*D3
- new net D5: U$7.P0[5], U1.*D5
- new net D6: U1.*D6
- new net D9: U$7.P0[6], U1.*D9
- new net GND: C1.1, C11.1, C12.2, C13.2, C14.2, C2.1, C3.1, C4.1, C5.2, C6.2, C7.1, C8.1, C9.1, JP1.4, MB0.P$1, MB1.P$1, R2.1, U$3.VSS, U$4.1, U$5.1, U$7.VSSA1, U$7.VSSA2, U$7.VSSA3, U$7.VSSD, U1.GND@0, U1.GND@1, U1.GND@2
- new net H-REF-CAP: C11.2, U$7.P2[4]
- new net HUMIDITY: U$3.FOUT, U$7.P2[3]
- new net MB0: MB0.P$2, R9.2, U$7.P0[0]
- new net MB1: MB1.P$2, R10.2, U$7.P0[1]
- new net MBLED0: R7.1, U$7.P0[2]
- new net MBLED1: R8.1, U$7.P0[4]
- new net N$10: R5.2, ULED2.C
- new net N$11: R6.2, ULED3.C
- new net N$12: MBLED0.C, R7.2
- new net N$13: MBLED1.C, R8.2
- new net N$14: U$2.VDD, U$4.2
- new net N$15: B3.BUTTON, R16.2
- new net N$17: U$2.GND, U$5.2
- new net N$2: B0.BUTTON, R13.2
- new net N$20: C7.2, U$7.VCCD
- new net N$5: B1.BUTTON, R14.2
- new net N$7: B2.BUTTON, R15.2
- new net N$8: R3.2, ULED0.C
- new net N$9: R4.2, ULED1.C
- new net P30: U$7.P3[0]
- new net P31: U$7.P3[1]
- new net P32: U$7.P3[2]
- new net POT: R2.2, U$7.P3[4], U1.A2
- new net SCL: U$2.SCL, U$7.P4[0]
- new net SCLK: JP1.2
- new net SDA: U$2.SDA, U$7.P4[1]
- new net SDAT: JP1.1
- new net THERM-LOW: R11.2, U$7.P3[6]
- new net THERM-MID: R1.1, R11.1, U$7.P3[5]
- new net THERM-REF-HIGH: R1.2, U$7.P1[3], U$7.P3[7]
- new net TIA_IN: ALS.C1, C10.1, R12.1, U$7.P2[1]
- new net TIA_OUT: C10.2, R12.2, R17.2, U$7.P2[2]
- new net UARTRX: U$7.P1[1], U1.TX
- new net UARTTX: U$7.P1[0], U1.RX
- new net V33: JMP1.3, JMP2.1, U1.3.3V
- new net V50: JMP1.1, JMP2.3, U1.5V
- new net VDAC: U$7.P1[2], U1.A1
- new net VPWR: ALS.E1, C1.2, C2.2, C3.2, C4.2, C5.1, C6.1, C8.2, C9.2, JMP1.2, JMP2.2, JP1.5, MBLED0.A, MBLED1.A, R10.1, R2.3, R9.1, U$4.3, U$5.3, U$7.VDDA1, U$7.VDDA2, U$7.VDDA3, U$7.VDDD, ULED0.A, ULED1.A, ULED2.A, ULED3.A
- new net VREF: C13.1, U$7.P2[7]
- new net XRES: JP1.3, U$7.XRES, U1.RES
Other:
- note added: "Flip RX/TX"

Commit message: routing complete
Connections:
- removed net SCLK: JP1.2
- removed net SDAT: JP1.1
- net MB0: now also JP1.1
- net MB1: now also JP1.2
Changed lines of the file:
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@@
 <label x="76.2" y="58.42" size="1.778" layer="95"/>
+</segment>
+<segment>
+<pinref part="JP1" gate="G$1" pin="1"/>
+<wire x1="-25.4" y1="106.68" x2="-10.16" y2="106.68" width="0.1524" layer="91"/>
+<label x="-22.86" y="106.68" size="1.778" layer="95"/>
 </segment>
 </net>
@@
 <wire x1="71.12" y1="60.96" x2="83.82" y2="60.96" width="0.1524" layer="91"/>
 <label x="76.2" y="60.96" size="1.778" layer="95"/>
+</segment>
+<segment>
+<pinref part="JP1" gate="G$1" pin="2"/>
+<wire x1="-25.4" y1="109.22" x2="-10.16" y2="109.22" width="0.1524" layer="91"/>
+<label x="-22.86" y="109.22" size="1.778" layer="95"/>
 </segment>
 </net>
@@
 </segment>
 </net>
-<net name="SDAT" class="0">
-<segment>
-<pinref part="JP1" gate="G$1" pin="1"/>
-<wire x1="-25.4" y1="106.68" x2="-10.16" y2="106.68" width="0.1524" layer="91"/>
-<label x="-22.86" y="106.68" size="1.778" layer="95"/>
-</segment>
-</net>
-<net name="SCLK" class="0">
-<segment>
-<pinref part="JP1" gate="G$1" pin="2"/>
-<wire x1="-25.4" y1="109.22" x2="-10.16" y2="109.22" width="0.1524" layer="91"/>
-<label x="-22.86" y="109.22" size="1.778" layer="95"/>
-</segment>
-</net>

Commit message: First complete board
Parts:
- removed JMP2: (no value), PatternAgents-ProtoPads:JMP-3-NO-0603
- added JPWR: 0, PatternAgents-ProtoPads:JMP-3-NO-0603
- added R18, R19, R20, R21: 10K, PatternAgents-ProtoPads:RESISTOR0603
- B0, B1, B2, B3: value (none) -> B
- C12: value (none) -> 2.2nF
- C13: value (none) -> 1uF
- C14: value (none) -> 10nF
- JMP1, JP1: value (none) -> 0
- MBLED0, MBLED1, ULED0, ULED1, ULED2, ULED3: value (none) -> red
- R1, R2: value (none) -> 10K
- renumbered ALS to D1, U$3 to HUMIDITY, U$4 to R30, U$5 to R31
Connections:
- removed net D6: U1.*D6
- removed net P30: U$7.P3[0]
- removed net P31: U$7.P3[1]
- removed net P32: U$7.P3[2]
- net GND: now also R30.3; no longer R30.1
- net SCL: now also R18.1, R19.1
- net SDA: now also R20.1, R21.1
- net V33: now also JPWR.3; no longer JMP2.1
- net V50: now also JPWR.1; no longer JMP2.3
- net VPWR: now also JPWR.2, R18.2, R19.2, R20.2, R21.2, R30.1; no longer JMP2.2, R30.3

Commit message: Fixed resistors
Parts:
- R3, R4, R5, R6, R7, R8: value 330 -> 560
Changed lines of the file:
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@@
 <part name="ULED2" library="adafruit" deviceset="LED" device="CHIP-LED0603" value="red"/>
 <part name="ULED3" library="adafruit" deviceset="LED" device="CHIP-LED0603" value="red"/>
-<part name="R3" library="PatternAgents-ProtoPads" deviceset="RESISTOR" device="0603" value="330"/>
-<part name="R4" library="PatternAgents-ProtoPads" deviceset="RESISTOR" device="0603" value="330"/>
-<part name="R5" library="PatternAgents-ProtoPads" deviceset="RESISTOR" device="0603" value="330"/>
-<part name="R6" library="PatternAgents-ProtoPads" deviceset="RESISTOR" device="0603" value="330"/>
-<part name="R7" library="PatternAgents-ProtoPads" deviceset="RESISTOR" device="0603" value="330"/>
-<part name="R8" library="PatternAgents-ProtoPads" deviceset="RESISTOR" device="0603" value="330"/>
+<part name="R3" library="PatternAgents-ProtoPads" deviceset="RESISTOR" device="0603" value="560"/>
+<part name="R4" library="PatternAgents-ProtoPads" deviceset="RESISTOR" device="0603" value="560"/>
+<part name="R5" library="PatternAgents-ProtoPads" deviceset="RESISTOR" device="0603" value="560"/>
+<part name="R6" library="PatternAgents-ProtoPads" deviceset="RESISTOR" device="0603" value="560"/>
+<part name="R7" library="PatternAgents-ProtoPads" deviceset="RESISTOR" device="0603" value="560"/>
+<part name="R8" library="PatternAgents-ProtoPads" deviceset="RESISTOR" device="0603" value="560"/>
 <part name="JMP1" library="PatternAgents-ProtoPads" deviceset="JMP-3-NO" device="-PTH" value="0"/>
 <part name="JPWR" library="PatternAgents-ProtoPads" deviceset="JMP-3-NO" device="-0603" value="0"/>

Commit message: Massive updates to the board
Parts:
- removed U1: ARDUINO_SHIELDNOHOLESORLABELS, SparkFun-Boards:ARDUINO_SHIELDNOHOLESORLABELS
- added U$1: ARDUINO_R3_SHIELDNOLABELS, SparkFun-Boards:ARDUINO_R3_SHIELDNOLABELS
- R18, R19, R20, R21: value 10K -> 4.7K
Connections:
- removed net THERM-LOW: R11.2, U$7.P3[6]
- net A0: now also U$1.A0; no longer U1.A0
- net D10: now also U$1.*D10; no longer U1.*D10
- net D3: now also U$1.*D3; no longer U1.*D3
- net D5: now also U$1.*D5; no longer U1.*D5
- net D9: now also U$1.*D9; no longer U1.*D9
- net GND: now also R11.2, U$1.GND@0, U$1.GND@1, U$1.GND@2, U$7.P3[7]; no longer U1.GND@0, U1.GND@1, U1.GND@2
- net POT: now also U$1.A2; no longer U1.A2
- net SCL: now also U$1.SCL
- net SDA: now also U$1.SDA
- net THERM-REF-HIGH: now also U$7.P3[6]; no longer U$7.P3[7]
- net UARTRX: now also U$1.TX; no longer U1.TX
- net UARTTX: now also U$1.RX; no longer U1.RX
- net V33: now also U$1.3.3V; no longer U1.3.3V
- net V50: now also U$1.5V; no longer U1.5V
- net VDAC: now also U$1.A1; no longer U1.A1
- net XRES: now also U$1.RES; no longer U1.RES
Changed lines of the file:
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@@
 <part name="C12" library="PatternAgents-ProtoPads" deviceset="CAP" device="0603-CAP" value="2.2nF"/>
 <part name="C13" library="PatternAgents-ProtoPads" deviceset="CAP" device="0603-CAP" value="1uF"/>
-<part name="U1" library="SparkFun-Boards" deviceset="ARDUINO_SHIELD" device="NOHOLESORLABELS"/>
 <part name="B0" library="PatternAgents-TouchWidgets" deviceset="BUTTON_PASSIVE" device="10MM" value="B"/>
 <part name="B1" library="PatternAgents-TouchWidgets" deviceset="BUTTON_PASSIVE" device="10MM" value="B"/>
@@
 <part name="B3" library="PatternAgents-TouchWidgets" deviceset="BUTTON_PASSIVE" device="10MM" value="B"/>
 <part name="C14" library="PatternAgents-ProtoPads" deviceset="CAP" device="0603-CAP" value="10nF"/>
-<part name="R18" library="PatternAgents-ProtoPads" deviceset="RESISTOR" device="0603" value="10K"/>
-<part name="R19" library="PatternAgents-ProtoPads" deviceset="RESISTOR" device="0603" value="10K"/>
-<part name="R20" library="PatternAgents-ProtoPads" deviceset="RESISTOR" device="0603" value="10K"/>
-<part name="R21" library="PatternAgents-ProtoPads" deviceset="RESISTOR" device="0603" value="10K"/>
+<part name="R18" library="PatternAgents-ProtoPads" deviceset="RESISTOR" device="0603" value="4.7K"/>
+<part name="R19" library="PatternAgents-ProtoPads" deviceset="RESISTOR" device="0603" value="4.7K"/>
+<part name="R20" library="PatternAgents-ProtoPads" deviceset="RESISTOR" device="0603" value="4.7K"/>
+<part name="R21" library="PatternAgents-ProtoPads" deviceset="RESISTOR" device="0603" value="4.7K"/>
+<part name="U$1" library="SparkFun-Boards" deviceset="ARDUINO_R3_SHIELD" device="NOLABELS"/>
 </parts>
 <sheets>
@@
 <instance part="R15" gate="R" x="137.16" y="147.32" rot="R180"/>
 <instance part="R16" gate="R" x="137.16" y="121.92" rot="R180"/>
-<instance part="U1" gate="G$1" x="55.88" y="172.72"/>
 <instance part="B0" gate="B1" x="116.84" y="198.12"/>
 <instance part="B1" gate="B1" x="116.84" y="172.72"/>
@@
 <instance part="R20" gate="R" x="58.42" y="109.22" rot="R180"/>
 <instance part="R21" gate="R" x="58.42" y="101.6" rot="R180"/>
+<instance part="U$1" gate="G$1" x="55.88" y="172.72"/>
 </instances>
 <busses>
@@
 </segment>
 <segment>
-<pinref part="U1" gate="G$1" pin="GND@2"/>
-<wire x1="43.18" y1="160.02" x2="33.02" y2="160.02" width="0.1524" layer="91"/>
-<wire x1="33.02" y1="160.02" x2="33.02" y2="157.48" width="0.1524" layer="91"/>
-<pinref part="U1" gate="G$1" pin="GND@1"/>
-<wire x1="33.02" y1="157.48" x2="43.18" y2="157.48" width="0.1524" layer="91"/>
-<pinref part="U1" gate="G$1" pin="GND@0"/>
 <wire x1="43.18" y1="154.94" x2="33.02" y2="154.94" width="0.1524" layer="91"/>
-<wire x1="33.02" y1="154.94" x2="33.02" y2="157.48" width="0.1524" layer="91"/>
-<label x="33.02" y="160.02" size="1.778" layer="95"/>
-<junction x="43.18" y="154.94"/>
-<junction x="43.18" y="157.48"/>
-<junction x="43.18" y="160.02"/>
-<junction x="33.02" y="160.02"/>
-<junction x="33.02" y="157.48"/>
+<pinref part="U$1" gate="G$1" pin="GND@2"/>
+<pinref part="U$1" gate="G$1" pin="GND@0"/>
+<wire x1="43.18" y1="149.86" x2="33.02" y2="149.86" width="0.1524" layer="91"/>
+<wire x1="33.02" y1="149.86" x2="33.02" y2="152.4" width="0.1524" layer="91"/>
+<pinref part="U$1" gate="G$1" pin="GND@1"/>
+<wire x1="33.02" y1="152.4" x2="33.02" y2="154.94" width="0.1524" layer="91"/>
+<wire x1="43.18" y1="152.4" x2="33.02" y2="152.4" width="0.1524" layer="91"/>
+<label x="33.02" y="154.94" size="1.778" layer="95"/>
+<junction x="33.02" y="149.86"/>
+<junction x="33.02" y="152.4"/>
 <junction x="33.02" y="154.94"/>
 </segment>
@@
 <wire x1="43.18" y1="185.42" x2="27.94" y2="185.42" width="0.1524" layer="91"/>
 <label x="27.94" y="185.42" size="1.778" layer="95"/>
-<pinref part="U1" gate="G$1" pin="A2"/>
+<pinref part="U$1" gate="G$1" pin="A2"/>
 </segment>
 </net>
@@
 <label x="66.04" y="109.22" size="1.778" layer="95"/>
 </segment>
+<segment>
+<pinref part="U$1" gate="G$1" pin="SDA"/>
+<wire x1="68.58" y1="152.4" x2="83.82" y2="152.4" width="0.1524" layer="91"/>
+<label x="73.66" y="152.4" size="1.778" layer="95"/>
+</segment>
 </net>
 <net name="N$17" class="0">
@@
 <label x="66.04" y="124.46" size="1.778" layer="95"/>
 </segment>
+<segment>
+<pinref part="U$1" gate="G$1" pin="SCL"/>
+<wire x1="68.58" y1="149.86" x2="83.82" y2="149.86" width="0.1524" layer="91"/>
+<label x="73.66" y="149.86" size="1.778" layer="95"/>
+</segment>
 </net>
 <net name="UARTRX" class="0">
@@
 <wire x1="68.58" y1="187.96" x2="83.82" y2="187.96" width="0.1524" layer="91"/>
 <label x="71.12" y="187.96" size="1.778" layer="95"/>
-<pinref part="U1" gate="G$1" pin="TX"/>
+<pinref part="U$1" gate="G$1" pin="TX"/>
 </segment>
 </net>
@@
 <wire x1="68.58" y1="190.5" x2="83.82" y2="190.5" width="0.1524" layer="91"/>
 <label x="71.12" y="190.5" size="1.778" layer="95"/>
-<pinref part="U1" gate="G$1" pin="RX"/>
+<pinref part="U$1" gate="G$1" pin="RX"/>
 </segment>
 </net>
@@
 <wire x1="68.58" y1="180.34" x2="83.82" y2="180.34" width="0.1524" layer="91"/>
 <label x="71.12" y="180.34" size="1.778" layer="95"/>
-<pinref part="U1" gate="G$1" pin="*D3"/>
+<pinref part="U$1" gate="G$1" pin="*D3"/>
 </segment>
 </net>
@@
 <wire x1="68.58" y1="175.26" x2="83.82" y2="175.26" width="0.1524" layer="91"/>
 <label x="71.12" y="175.26" size="1.778" layer="95"/>
-<pinref part="U1" gate="G$1" pin="*D5"/>
+<pinref part="U$1" gate="G$1" pin="*D5"/>
 </segment>
 </net>
@@
 <wire x1="68.58" y1="165.1" x2="86.36" y2="165.1" width="0.1524" layer="91"/>
 <label x="73.66" y="165.1" size="1.778" layer="95"/>
-<pinref part="U1" gate="G$1" pin="*D9"/>
+<pinref part="U$1" gate="G$1" pin="*D9"/>
 </segment>
 </net>
@@
 <wire x1="68.58" y1="162.56" x2="83.82" y2="162.56" width="0.1524" layer="91"/>
 <label x="71.12" y="162.56" size="1.778" layer="95"/>
-<pinref part="U1" gate="G$1" pin="*D10"/>
+<pinref part="U$1" gate="G$1" pin="*D10"/>
 </segment>
 </net>
@@
 <wire x1="43.18" y1="190.5" x2="27.94" y2="190.5" width="0.1524" layer="91"/>
 <label x="27.94" y="190.5" size="1.778" layer="95"/>
-<pinref part="U1" gate="G$1" pin="A0"/>
+<pinref part="U$1" gate="G$1" pin="A0"/>
 </segment>
 </net>
@@
 <wire x1="43.18" y1="187.96" x2="27.94" y2="187.96" width="0.1524" layer="91"/>
 <label x="27.94" y="187.96" size="1.778" layer="95"/>
-<pinref part="U1" gate="G$1" pin="A1"/>
+<pinref part="U$1" gate="G$1" pin="A1"/>
+</segment>
+</net>
+<net name="XRES" class="0">
+<segment>
+<pinref part="U$1" gate="G$1" pin="RES"/>
+<wire x1="43.18" y1="167.64" x2="30.48" y2="167.64" width="0.1524" layer="91"/>
+<label x="30.48" y="167.64" size="1.778" layer="95"/>
+</segment>
+</net>
+<net name="V33" class="0">
+<segment>
+<pinref part="U$1" gate="G$1" pin="3.3V"/>
+<wire x1="43.18" y1="160.02" x2="33.02" y2="160.02" width="0.1524" layer="91"/>
+<label x="33.02" y="160.02" size="1.778" layer="95"/>
 </segment>
 </net>
 <net name="V50" class="0">
 <segment>
-<pinref part="U1" gate="G$1" pin="5V"/>
-<wire x1="43.18" y1="167.64" x2="33.02" y2="167.64" width="0.1524" layer="91"/>
-<label x="33.02" y="167.64" size="1.778" layer="95"/>
-</segment>
-</net>
-<net name="XRES" class="0">
-<segment>
-<pinref part="U1" gate="G$1" pin="RES"/>
-<wire x1="43.18" y1="172.72" x2="33.02" y2="172.72" width="0.1524" layer="91"/>
-<label x="33.02" y="172.72" size="1.778" layer="95"/>
-</segment>
-</net>
-<net name="V33" class="0">
-<segment>
-<pinref part="U1" gate="G$1" pin="3.3V"/>
-<wire x1="43.18" y1="165.1" x2="33.02" y2="165.1" width="0.1524" layer="91"/>
-<label x="33.02" y="165.1" size="1.778" layer="95"/>
+<pinref part="U$1" gate="G$1" pin="5V"/>
+<wire x1="43.18" y1="162.56" x2="33.02" y2="162.56" width="0.1524" layer="91"/>
+<label x="33.02" y="162.56" size="1.778" layer="95"/>
 </segment>
 </net>
@@
 </segment>
 </net>
-<net name="THERM-LOW" class="0">
+<net name="THERM-REF-HIGH" class="0">
+<segment>
+<pinref part="U$7" gate="G$1" pin="P1[3]"/>
+<wire x1="7.62" y1="73.66" x2="-5.08" y2="73.66" width="0.1524" layer="91"/>
+<label x="-2.54" y="73.66" size="1.778" layer="95"/>
+</segment>
 <segment>
 <pinref part="U$7" gate="G$1" pin="P3[6]"/>
 <wire x1="71.12" y1="53.34" x2="83.82" y2="53.34" width="0.1524" layer="91"/>
 <label x="76.2" y="53.34" size="1.778" layer="95"/>
-</segment>
-</net>
-<net name="THERM-REF-HIGH" class="0">
-<segment>
-<pinref part="U$7" gate="G$1" pin="P3[7]"/>
-<wire x1="71.12" y1="55.88" x2="83.82" y2="55.88" width="0.1524" layer="91"/>
-<label x="76.2" y="55.88" size="1.778" layer="95"/>
-</segment>
-<segment>
-<pinref part="U$7" gate="G$1" pin="P1[3]"/>
-<wire x1="7.62" y1="73.66" x2="-5.08" y2="73.66" width="0.1524" layer="91"/>
-<label x="-2.54" y="73.66" size="1.778" layer="95"/>
 </segment>
 </net>
@@
 <wire x1="40.64" y1="15.24" x2="40.64" y2="20.32" width="0.1524" layer="91"/>
 <label x="35.56" y="15.24" size="1.778" layer="95" rot="R90"/>
+</segment>
+<segment>
+<pinref part="U$7" gate="G$1" pin="P3[7]"/>
+<wire x1="71.12" y1="55.88" x2="83.82" y2="55.88" width="0.1524" layer="91"/>
+<label x="76.2" y="55.88" size="1.778" layer="95"/>
 </segment>
 </net>
@@
 </segment>
 </net>
-<net name="THERM-LOW" class="0">
-<segment>
-<pinref part="R11" gate="G$1" pin="2"/>
-<wire x1="99.06" y1="91.44" x2="99.06" y2="86.36" width="0.1524" layer="91"/>
-<wire x1="99.06" y1="86.36" x2="88.9" y2="86.36" width="0.1524" layer="91"/>
-<label x="88.9" y="86.36" size="1.778" layer="95"/>
-</segment>
-</net>
 <net name="TIA_IN" class="0">
 <segment>
@@
 <label x="5.08" y="144.78" size="1.778" layer="95"/>
 </segment>
+<segment>
+<pinref part="R11" gate="G$1" pin="2"/>
+<wire x1="99.06" y1="91.44" x2="99.06" y2="86.36" width="0.1524" layer="91"/>
+<wire x1="99.06" y1="86.36" x2="88.9" y2="86.36" width="0.1524" layer="91"/>
+<label x="88.9" y="86.36" size="1.778" layer="95"/>
+</segment>
 </net>
 <net name="HUMIDITY" class="0">
@@
 </sheet>
 </sheets>
+<errors>
+</errors>
 </schematic>
 </drawing>
