File: ww101-shield/eagle/ww101board.sch (EAGLE design)
At the start: 57 parts

Commit message: Right before autoroute
Parts:
- added LED2: red, adafruit:LEDCHIP-LED0603
- added R22: 10K, PatternAgents-ProtoPads:RESISTOR0603
- added R23: 560, PatternAgents-ProtoPads:RESISTOR0603
- renumbered MB0 to MB2
Connections:
- net MBLED1 renamed LED1
- removed net D10: U$1.*D10, U$7.P0[7]
- removed net D3: U$1.*D3, U$7.P0[3]
- removed net D9: U$1.*D9, U$7.P0[6]
- removed net MB0: JP1.2, MB2.P$2, R10.2, U$7.P0[1]
- removed net MBLED0: R7.1, U$7.P0[2]
- new net D11: U$1.*D11, U$7.P0[7]
- new net D12: U$1.D12, U$7.P0[2]
- new net D13: U$1.D13, U$7.P3[1]
- new net D4: U$1.D4, U$7.P0[3]
- new net FUTUREARD: U$1.D2, U$7.P3[2]
- new net LED2: R7.1, U$7.P0[6]
- new net MB2: JP1.1, MB2.P$2, R10.2, U$7.P0[0]
- new net N$3: LED2.C, R23.2
- new net PROXLED: R23.1, U$7.P3[0]
- net MB1: now also JP1.2, U$7.P0[1]; no longer JP1.1, U$7.P0[0]
- net VPWR: now also LED2.A, R22.1
- net XRES: now also R22.2
Other:
- note added: "SCLK"
- note added: "SDAT"

Commit message: V2.0 of board
Parts:
- removed LED0: red, adafruit:LEDCHIP-LED0603
- added PROX: red, adafruit:LEDCHIP-LED0603
- added R24: 0R, PatternAgents-ProtoPads:RESISTOR0603
Connections:
- new net CMESH: R24.1
- net CSHIELD: now also R24.2
- net LED1: now also R7.1, U$7.P0[6]; no longer R8.1, U$7.P0[4]
- net LED2: now also R8.1, U$7.P0[4]; no longer R7.1, U$7.P0[6]
- net MB1: now also JP1.1, R10.2, U$7.P0[0]; no longer JP1.2, R9.2, U$7.P0[1]
- net MB2: now also JP1.2, R9.2, U$7.P0[1]; no longer JP1.1, R10.2, U$7.P0[0]
- net N$12: now also LED1.C; no longer LED0.C
- net N$13: now also LED2.C; no longer LED1.C
- net N$3: now also PROX.C; no longer LED2.C
- net VPWR: now also PROX.A; no longer LED0.A
Other:
- note added: "1%"
- moved on the sheet: LED1, LED2, MB1, MB2
Changed lines of the file:
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@@
 <parts>
 <part name="U$2" library="IOTExpert" deviceset="U8G-096-OLED" device=""/>
+<part name="MB2" library="IOTExpert" deviceset="EVQPE1" device=""/>
 <part name="MB1" library="IOTExpert" deviceset="EVQPE1" device=""/>
-<part name="MB2" library="IOTExpert" deviceset="EVQPE1" device=""/>
 <part name="U$7" library="PatternAgents-Cypress" deviceset="CY8C4A45-48" device=""/>
 <part name="C1" library="PatternAgents-ProtoPads" deviceset="CAP" device="0603-CAP" value="1uF"/>
@@
 <part name="C9" library="PatternAgents-ProtoPads" deviceset="CAP" device="0603-CAP" value="0.1uF"/>
 <part name="R2" library="pot" deviceset="TRIM_US-" device="3386P" value="10K"/>
-<part name="LED0" library="adafruit" deviceset="LED" device="CHIP-LED0603" value="red"/>
 <part name="LED1" library="adafruit" deviceset="LED" device="CHIP-LED0603" value="red"/>
+<part name="LED2" library="adafruit" deviceset="LED" device="CHIP-LED0603" value="red"/>
 <part name="CLED0" library="adafruit" deviceset="LED" device="CHIP-LED0603" value="red"/>
 <part name="CLED1" library="adafruit" deviceset="LED" device="CHIP-LED0603" value="red"/>
@@
 <part name="U$1" library="SparkFun-Boards" deviceset="ARDUINO_R3_SHIELD" device="NOLABELS"/>
 <part name="R22" library="PatternAgents-ProtoPads" deviceset="RESISTOR" device="0603" value="10K"/>
-<part name="LED2" library="adafruit" deviceset="LED" device="CHIP-LED0603" value="red"/>
+<part name="PROX" library="adafruit" deviceset="LED" device="CHIP-LED0603" value="red"/>
 <part name="R23" library="PatternAgents-ProtoPads" deviceset="RESISTOR" device="0603" value="560"/>
+<part name="R24" library="PatternAgents-ProtoPads" deviceset="RESISTOR" device="0603" value="0R"/>
 </parts>
 <sheets>
@@
 <instances>
 <instance part="U$2" gate="G$1" x="114.3" y="53.34"/>
-<instance part="MB1" gate="G$1" x="124.46" y="78.74"/>
-<instance part="MB2" gate="G$1" x="124.46" y="88.9"/>
+<instance part="MB2" gate="G$1" x="124.46" y="78.74"/>
+<instance part="MB1" gate="G$1" x="124.46" y="88.9"/>
 <instance part="R2" gate="1" x="149.86" y="53.34"/>
-<instance part="LED0" gate="G$1" x="187.96" y="88.9" rot="R90"/>
-<instance part="LED1" gate="G$1" x="187.96" y="76.2" rot="R90"/>
+<instance part="LED1" gate="G$1" x="187.96" y="88.9" rot="R90"/>
+<instance part="LED2" gate="G$1" x="187.96" y="76.2" rot="R90"/>
 <instance part="CLED0" gate="G$1" x="190.5" y="198.12" rot="R90"/>
 <instance part="CLED1" gate="G$1" x="190.5" y="172.72" rot="R90"/>
@@
 <instance part="R21" gate="R" x="58.42" y="101.6" rot="R180"/>
 <instance part="U$1" gate="G$1" x="55.88" y="172.72"/>
-<instance part="LED2" gate="G$1" x="187.96" y="55.88" rot="R90"/>
+<instance part="PROX" gate="G$1" x="187.96" y="55.88" rot="R90"/>
 <instance part="R23" gate="R" x="198.12" y="55.88" rot="R180"/>
 </instances>
@@
 <segment>
 <wire x1="185.42" y1="76.2" x2="185.42" y2="83.82" width="0.1524" layer="91"/>
-<pinref part="LED0" gate="G$1" pin="A"/>
 <pinref part="LED1" gate="G$1" pin="A"/>
+<pinref part="LED2" gate="G$1" pin="A"/>
 <wire x1="185.42" y1="83.82" x2="185.42" y2="88.9" width="0.1524" layer="91"/>
 <wire x1="185.42" y1="83.82" x2="175.26" y2="83.82" width="0.1524" layer="91"/>
@@
 </segment>
 <segment>
-<pinref part="LED2" gate="G$1" pin="A"/>
+<pinref part="PROX" gate="G$1" pin="A"/>
 <wire x1="185.42" y1="55.88" x2="175.26" y2="55.88" width="0.1524" layer="91"/>
 <label x="175.26" y="55.88" size="1.778" layer="95"/>
@@
 </segment>
 </net>
-<net name="MB1" class="0">
-<segment>
-<pinref part="MB1" gate="G$1" pin="P$2"/>
-<pinref part="R9" gate="R" pin="2"/>
-<wire x1="149.86" y1="78.74" x2="134.62" y2="78.74" width="0.1524" layer="91"/>
-<label x="139.7" y="78.74" size="1.778" layer="95"/>
-</segment>
-</net>
 <net name="GND" class="0">
 <segment>
-<pinref part="MB1" gate="G$1" pin="P$1"/>
+<pinref part="MB2" gate="G$1" pin="P$1"/>
 <wire x1="124.46" y1="78.74" x2="119.38" y2="78.74" width="0.1524" layer="91"/>
 <wire x1="119.38" y1="78.74" x2="119.38" y2="88.9" width="0.1524" layer="91"/>
-<pinref part="MB2" gate="G$1" pin="P$1"/>
+<pinref part="MB1" gate="G$1" pin="P$1"/>
 <wire x1="119.38" y1="88.9" x2="124.46" y2="88.9" width="0.1524" layer="91"/>
 <label x="119.38" y="91.44" size="1.778" layer="95" rot="R90"/>
@@
 </segment>
 </net>
-<net name="MB2" class="0">
-<segment>
-<pinref part="MB2" gate="G$1" pin="P$2"/>
-<pinref part="R10" gate="R" pin="2"/>
-<wire x1="134.62" y1="88.9" x2="149.86" y2="88.9" width="0.1524" layer="91"/>
-<label x="137.16" y="88.9" size="1.778" layer="95"/>
-</segment>
-</net>
 <net name="N$12" class="0">
 <segment>
-<pinref part="LED0" gate="G$1" pin="C"/>
+<pinref part="LED1" gate="G$1" pin="C"/>
 <pinref part="R7" gate="R" pin="2"/>
 </segment>
@@
 <net name="N$13" class="0">
 <segment>
-<pinref part="LED1" gate="G$1" pin="C"/>
+<pinref part="LED2" gate="G$1" pin="C"/>
 <pinref part="R8" gate="R" pin="2"/>
 </segment>
@@
 <net name="N$3" class="0">
 <segment>
-<pinref part="LED2" gate="G$1" pin="C"/>
+<pinref part="PROX" gate="G$1" pin="C"/>
 <pinref part="R23" gate="R" pin="2"/>
 </segment>
@@
 </segment>
 </net>
-<net name="LED2" class="0">
+<net name="LED1" class="0">
 <segment>
 <pinref part="R7" gate="R" pin="1"/>
@@
 </segment>
 </net>
-<net name="LED1" class="0">
+<net name="LED2" class="0">
 <segment>
 <pinref part="R8" gate="R" pin="1"/>
@@
 <wire x1="68.58" y1="154.94" x2="83.82" y2="154.94" width="0.1524" layer="91"/>
 <label x="73.66" y="154.94" size="1.778" layer="95"/>
+</segment>
+</net>
+<net name="MB1" class="0">
+<segment>
+<pinref part="MB1" gate="G$1" pin="P$2"/>
+<pinref part="R10" gate="R" pin="2"/>
+<wire x1="134.62" y1="88.9" x2="149.86" y2="88.9" width="0.1524" layer="91"/>
+<label x="137.16" y="88.9" size="1.778" layer="95"/>
+</segment>
+</net>
+<net name="MB2" class="0">
+<segment>
+<pinref part="MB2" gate="G$1" pin="P$2"/>
+<pinref part="R9" gate="R" pin="2"/>
+<wire x1="134.62" y1="78.74" x2="149.86" y2="78.74" width="0.1524" layer="91"/>
+<label x="137.16" y="78.74" size="1.778" layer="95"/>
 </segment>
 </net>
@@
 <instance part="C14" gate="G$1" x="-40.64" y="88.9"/>
 <instance part="R22" gate="R" x="73.66" y="121.92" rot="R180"/>
+<instance part="R24" gate="R" x="63.5" y="22.86" rot="R180"/>
 </instances>
 <busses>
@@
 <net name="MB1" class="0">
 <segment>
-<pinref part="U$7" gate="G$1" pin="P0[1]"/>
-<wire x1="71.12" y1="60.96" x2="83.82" y2="60.96" width="0.1524" layer="91"/>
-<label x="76.2" y="60.96" size="1.778" layer="95"/>
-</segment>
-<segment>
-<pinref part="JP1" gate="G$1" pin="2"/>
-<wire x1="-25.4" y1="109.22" x2="-10.16" y2="109.22" width="0.1524" layer="91"/>
-<label x="-22.86" y="109.22" size="1.778" layer="95"/>
-</segment>
-</net>
-<net name="MB2" class="0">
+<pinref part="JP1" gate="G$1" pin="1"/>
+<wire x1="-25.4" y1="106.68" x2="-10.16" y2="106.68" width="0.1524" layer="91"/>
+<label x="-22.86" y="106.68" size="1.778" layer="95"/>
+</segment>
 <segment>
 <pinref part="U$7" gate="G$1" pin="P0[0]"/>
@@
 <label x="76.2" y="58.42" size="1.778" layer="95"/>
 </segment>
-<segment>
-<pinref part="JP1" gate="G$1" pin="1"/>
-<wire x1="-25.4" y1="106.68" x2="-10.16" y2="106.68" width="0.1524" layer="91"/>
-<label x="-22.86" y="106.68" size="1.778" layer="95"/>
-</segment>
 </net>
 <net name="D12" class="0">
@@
 </segment>
 </net>
-<net name="LED1" class="0">
+<net name="LED2" class="0">
 <segment>
 <pinref part="U$7" gate="G$1" pin="P0[4]"/>
@@
 <segment>
 <pinref part="U$7" gate="G$1" pin="P3[3]"/>
-<wire x1="50.8" y1="40.64" x2="50.8" y2="30.48" width="0.1524" layer="91"/>
+<wire x1="50.8" y1="40.64" x2="50.8" y2="22.86" width="0.1524" layer="91"/>
 <label x="50.8" y="30.48" size="1.778" layer="95" rot="R90"/>
+<pinref part="R24" gate="R" pin="2"/>
+<wire x1="50.8" y1="22.86" x2="58.42" y2="22.86" width="0.1524" layer="91"/>
 </segment>
 </net>
@@
 </segment>
 </net>
-<net name="LED2" class="0">
+<net name="LED1" class="0">
 <segment>
 <pinref part="U$7" gate="G$1" pin="P0[6]"/>
@@
 <wire x1="71.12" y1="76.2" x2="83.82" y2="76.2" width="0.1524" layer="91"/>
 <label x="76.2" y="76.2" size="1.778" layer="95"/>
+</segment>
+</net>
+<net name="MB2" class="0">
+<segment>
+<pinref part="U$7" gate="G$1" pin="P0[1]"/>
+<wire x1="71.12" y1="60.96" x2="83.82" y2="60.96" width="0.1524" layer="91"/>
+<label x="76.2" y="60.96" size="1.778" layer="95"/>
+</segment>
+<segment>
+<pinref part="JP1" gate="G$1" pin="2"/>
+<wire x1="-25.4" y1="109.22" x2="-10.16" y2="109.22" width="0.1524" layer="91"/>
+<label x="-22.86" y="109.22" size="1.778" layer="95"/>
+</segment>
+</net>
+<net name="CMESH" class="0">
+<segment>
+<pinref part="R24" gate="R" pin="1"/>
+<wire x1="68.58" y1="22.86" x2="76.2" y2="22.86" width="0.1524" layer="91"/>
+<label x="71.12" y="22.86" size="1.778" layer="95"/>
 </segment>
 </net>
@@
 <description>Sensor</description>
 <plain>
+<text x="43.18" y="149.86" size="1.778" layer="95" rot="R90">1% </text>
 </plain>
 <instances>

Commit message: before library update
Parts:
- added C15, C16, C17: 0.1uF, PatternAgents-ProtoPads:CAP0603-CAP
- added R25: 0R, PatternAgents-ProtoPads:RESISTOR0603
Connections:
- removed net VPWR: C1.2, C2.2, C3.2, C4.2, C5.1, C6.1, C8.2, C9.2, CLED0.A, CLED1.A, CLED2.A, CLED3.A, D1.E1, JMP1.2, JP1.5, JPWR.2, LED1.A, LED2.A, PROX.A, R10.1, R18.2, R19.2, R2.3, R20.2, R21.2, R22.1, R30.1, R31.3, R9.1, U$7.VDDA1, U$7.VDDA2, U$7.VDDA3, U$7.VDDD
- new net CAP-PSOC: R25.2, U$7.P2[5]
- new net VCC: C1.2, C15.1, C17.1, C2.2, C3.2, C4.2, C5.1, C6.1, C8.2, C9.2, CLED0.A, CLED1.A, CLED2.A, CLED3.A, D1.E1, JMP1.2, JP1.5, JPWR.2, LED1.A, LED2.A, PROX.A, R10.1, R18.2, R19.2, R2.3, R20.2, R21.2, R22.1, R30.1, R31.3, R9.1, U$7.VDDA1, U$7.VDDA2, U$7.VDDA3, U$7.VDDD
- net CAP-PROX: now also R25.1; no longer U$7.P2[5]
- net GND: now also C16.2, C17.2
- net POT: now also C16.1
- net XRES: now also C15.2
Other:
- note added: "PSoC"
- note added: "Power"
- note added: "Sensors"
- note added: "User Interface"
- moved on the sheet: B0, B1, B2, B3, C12, C13, C14, C5, C6, C7, C8, C9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

Commit message: the saturday night checkin of all of the V2.1 changes
Parts:
- removed JMP1: 0, PatternAgents-ProtoPads:JMP-3-NO-PTH
- removed JP1: 0, SparkFun-Connectors:M05LOCK
- removed JPWR: 0, PatternAgents-ProtoPads:JMP-3-NO-0603
- removed U$2: U8G-096-OLED, IOTExpert:U8G-096-OLED
- added J5: (no value), ww101board:JMP-3-PTH-PTH
- added J6: U8G-096-OLED, ww101board:U8G-096-OLED
- added J7: 0, ww101board:M05LOCK
- added R32: (no value), ww101board:JMP-3-NO
- B0, B1, B2, B3: device PatternAgents-TouchWidgets:BUTTON_PASSIVE10MM -> ww101board:BUTTON_PASSIVE10MM
- C1, C10, C11, C12, C13, C14, C15, C16, C17, C2, C3, C4, C5, C6, C7, C8, C9: device PatternAgents-ProtoPads:CAP0603-CAP -> ww101board:CAP0603-CAP
- CLED0, CLED1, CLED2, CLED3, LED1, LED2, PROX: device adafruit:LEDCHIP-LED0603 -> ww101board:LEDCHIP-LED0603
- D1: device IOTExpert:ALS -> ww101board:ALS
- HUMIDITY: device IOTExpert:HPP801A031 -> ww101board:HPP801A031
- MB1, MB2: device IOTExpert:EVQPE1 -> ww101board:EVQPE1
- R1, R10, R12, R13, R14, R15, R16, R17, R18, R19, R20, R21, R22, R23, R24, R25, R3, R4, R5, R6, R7, R8, R9: device PatternAgents-ProtoPads:RESISTOR0603 -> ww101board:RESISTOR0603
- R11: device varistor:THERMISTOR-5 -> ww101board:THERMISTOR-5
- R2: device pot:TRIM_US-3386P -> ww101board:TRIM_US-3386P
- R30: device PatternAgents-ProtoPads:JMP-3-1_2 -> ww101board:JMP-3-1_2
- R31: device PatternAgents-ProtoPads:JMP-3-2_3 -> ww101board:JMP-3-2_3
- U$1: device SparkFun-Boards:ARDUINO_R3_SHIELDNOLABELS -> ww101board:ARDUINO_R3_SHIELDNOLABELS
- U$7: device PatternAgents-Cypress:CY8C4A45-48 -> ww101board:CY8C4A45-48
Connections:
- net GND: now also J7.4; no longer JP1.4
- net MB1: now also J7.1; no longer JP1.1
- net MB2: now also J7.2; no longer JP1.2
- net N$14: now also J6.VDD; no longer U$2.VDD
- net N$17: now also J6.GND; no longer U$2.GND
- net SCL: now also J6.SCL; no longer U$2.SCL
- net SDA: now also J6.SDA; no longer U$2.SDA
- net V33: now also J5.3, R32.1; no longer JMP1.3, JPWR.3
- net V50: now also J5.1, R32.3; no longer JMP1.1, JPWR.1
- net VCC: now also J5.2, J7.5, R32.2; no longer JMP1.2, JP1.5, JPWR.2
- net XRES: now also J7.3; no longer JP1.3
Other:
- note added: "10K"
- note added: "2.1"
- note added: "CY8C4247AZI-M485"
- note added: "DNP - J5 It will only be used in the situation where the user has to switch back and forth between v50 and v33 If that is required they will hand solder a header into the board and remove the 0ohm resistor from R32"
- note added: "J6"
- note added: "PSoC Analog CoProcessor"
- note added: "R32 is a 0 OHM resistor used to selec the power supply Please solder a 0 ohm into the 3.3V default position"
- note added: "The OLED Screen vendors sometimes have gnd/power and sometimes have power/gnd. R30 & R31 are 0 Ohm resistors on the top and bottom of the board let you select the screen type When assembling make sure you put them in the right place or they will be hard to fix!! If there is any doubt put them on the bottom of the board!!"
- note added: "Two sets of I2C Resistors (Top/Bottom) No Load - Only for base boards with no I2C resitors preinstalled on I2C"
- note removed: "PSoC"

Commit message: a bunch of minor tweaks
Parts:
- C17: value 0.1uF -> 10uF
- renumbered U$7 to U7
Other:
- note added: "R32 is a 0 OHM resistor used to select the power supply Please solder a 0 ohm into the 3.3V default position"
- note removed: "R32 is a 0 OHM resistor used to selec the power supply Please solder a 0 ohm into the 3.3V default position"

Commit message: a bunch of updates
Parts:
- added U$7: CYLOGO-SILK, ww101board:CYLOGO-SILK
- R18, R19, R20, R21: value 4.7K -> DNP
Other:
- note added: "CY8CKIT-032"
- note added: "PSoC"
- note added: "The OLED Screen vendors sometimes have gnd/power and sometimes have power/gnd. R30 & R31 are 0 Ohm resistors on the top of the board let you select the screen type When assembling make sure you put them in the right place or they will be hard to fix!! If there is any doubt put them on the bottom of the board!!"
- note removed: "PSoC Analog CoProcessor"
- note removed: "The OLED Screen vendors sometimes have gnd/power and sometimes have power/gnd. R30 & R31 are 0 Ohm resistors on the top and bottom of the board let you select the screen type When assembling make sure you put them in the right place or they will be hard to fix!! If there is any doubt put them on the bottom of the board!!"
Changed lines of the file:
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@@
 <layer number="155" name="FabDoc3" color="7" fill="1" visible="no" active="yes"/>
 <layer number="199" name="Contour" color="7" fill="1" visible="no" active="yes"/>
-<layer number="200" name="200bmp" color="1" fill="10" visible="no" active="yes"/>
+<layer number="200" name="200bmp" color="1" fill="10" visible="yes" active="yes"/>
 <layer number="201" name="201bmp" color="2" fill="10" visible="no" active="yes"/>
 <layer number="202" name="202bmp" color="3" fill="10" visible="no" active="yes"/>
@@
 <part name="B3" library="ww101board" deviceset="BUTTON_PASSIVE" device="10MM" value="B"/>
 <part name="C14" library="ww101board" deviceset="CAP" device="0603-CAP" value="10nF"/>
-<part name="R18" library="ww101board" deviceset="RESISTOR" device="0603" value="4.7K"/>
-<part name="R19" library="ww101board" deviceset="RESISTOR" device="0603" value="4.7K"/>
-<part name="R20" library="ww101board" deviceset="RESISTOR" device="0603" value="4.7K"/>
-<part name="R21" library="ww101board" deviceset="RESISTOR" device="0603" value="4.7K"/>
+<part name="R18" library="ww101board" deviceset="RESISTOR" device="0603" value="DNP"/>
+<part name="R19" library="ww101board" deviceset="RESISTOR" device="0603" value="DNP"/>
+<part name="R20" library="ww101board" deviceset="RESISTOR" device="0603" value="DNP"/>
+<part name="R21" library="ww101board" deviceset="RESISTOR" device="0603" value="DNP"/>
 <part name="R22" library="ww101board" deviceset="RESISTOR" device="0603" value="10K"/>
 <part name="PROX" library="ww101board" deviceset="LED" device="CHIP-LED0603" value="red"/>
@@
 <part name="J5" library="ww101board" deviceset="JMP-3-PTH" device="-PTH"/>
 <part name="R32" library="ww101board" deviceset="JMP-3-NO" device=""/>
+<part name="U$2" library="ww101board" deviceset="CYLOGO" device=""/>
+<part name="U$4" library="ww101board" deviceset="CYLOGO" device=""/>
+<part name="U$5" library="ww101board" deviceset="CYLOGO" device=""/>
+<part name="U$6" library="ww101board" deviceset="CYLOGO" device=""/>
+<part name="U$7" library="ww101board" deviceset="CYLOGO-SILK" device=""/>
 </parts>
 <sheets>
@@
 <plain>
 <text x="68.58" y="195.58" size="1.778" layer="95">Flip RX/TX</text>
-<text x="190.5" y="30.48" size="5.08" layer="97">User Interface</text>
+<text x="223.52" y="12.7" size="3.048" layer="97">User Interface</text>
 <text x="33.02" y="88.9" size="1.778" layer="97">Two sets of I2C Resistors (Top/Bottom)
 No Load - Only for base boards with
@@
 have gnd/power and sometimes have
 power/gnd.  R30 &amp; R31 are 0 Ohm
-resistors on the top and bottom of
-the board let you select the screen type
+resistors on the top of the board let
+you select the screen type
 When assembling make sure you put
 them in the right place or they will be
@@
 <text x="269.24" y="10.16" size="1.778" layer="97">2.1</text>
 <text x="76.2" y="45.72" size="1.778" layer="97">J6</text>
+<text x="236.22" y="30.48" size="3.81" layer="97">CY8CKIT-032</text>
 </plain>
 <instances>
@@
 <instance part="SUPPLY13" gate="GND" x="83.82" y="152.4" rot="R90"/>
 <instance part="U$1" gate="G$1" x="50.8" y="172.72"/>
+<instance part="U$2" gate="G$1" x="190.5" y="25.4"/>
 </instances>
 <busses>
@@
 <text x="-20.32" y="147.32" size="1.778" layer="97">SCLK</text>
 <text x="-20.32" y="144.78" size="1.778" layer="97">SDAT</text>
-<text x="68.58" y="5.08" size="4.826" layer="97">PSoC Analog CoProcessor</text>
+<text x="116.84" y="-12.7" size="3.048" layer="97">PSoC</text>
 <text x="157.48" y="-15.24" size="1.778" layer="97">2.1</text>
 <text x="27.94" y="66.04" size="1.778" layer="97">CY8C4247AZI-M485</text>
+<text x="121.92" y="5.08" size="3.81" layer="97">CY8CKIT-032</text>
 </plain>
 <instances>
@@
 </instance>
 <instance part="R25" gate="R" x="22.86" y="17.78"/>
+<instance part="U$4" gate="G$1" x="73.66" y="0"/>
+<instance part="U$7" gate="G$1" x="111.76" y="167.64"/>
 </instances>
 <busses>
@@
 <description>Power</description>
 <plain>
-<text x="132.08" y="68.58" size="5.08" layer="97">Power</text>
+<text x="170.18" y="50.8" size="5.08" layer="97">Power</text>
 <text x="215.9" y="50.8" size="1.778" layer="97">2.1</text>
 <text x="53.34" y="162.56" size="1.778" layer="97">DNP - J5
@@
 Please solder a 0 ohm into the 3.3V
 default position</text>
+<text x="182.88" y="71.12" size="3.81" layer="97">CY8CKIT-032</text>
 </plain>
 <instances>
@@
 <instance part="J5" gate="JMP" x="73.66" y="149.86"/>
 <instance part="R32" gate="G$1" x="96.52" y="149.86" rot="R180"/>
+<instance part="U$5" gate="G$1" x="139.7" y="66.04"/>
 </instances>
 <busses>
@@
 <plain>
 <text x="43.18" y="149.86" size="1.778" layer="95" rot="R90">1% </text>
-<text x="129.54" y="25.4" size="5.08" layer="97">Sensors</text>
+<text x="170.18" y="5.08" size="5.08" layer="97">Sensors</text>
 <text x="104.14" y="93.98" size="1.778" layer="97" rot="R90">10K</text>
 <text x="134.62" y="71.12" size="1.778" layer="97" rot="R180">2.1</text>
 <text x="220.98" y="7.62" size="1.778" layer="97" rot="R180">2.1</text>
+<text x="180.34" y="25.4" size="3.81" layer="97">CY8CKIT-032</text>
 </plain>
 <instances>
@@
 <attribute name="VALUE" x="182.499" y="133.604" size="1.778" layer="96" rot="R90"/>
 </instance>
+<instance part="U$6" gate="G$1" x="132.08" y="20.32"/>
 </instances>
 <busses>

Commit message: updates to 2.1 board based on GJL inputs
Other:
- note added: "P37 should be a direct path to thermistor ground"
- note added: "The OLED Screen vendors sometimes have gnd/power and sometimes have power/gnd. R30 & R31 are 0 Ohm resistors on the top of the board that let you select the screen type When assembling make sure you put them in the right place or they will be hard to fix!!"
- note removed: "The OLED Screen vendors sometimes have gnd/power and sometimes have power/gnd. R30 & R31 are 0 Ohm resistors on the top of the board let you select the screen type When assembling make sure you put them in the right place or they will be hard to fix!! If there is any doubt put them on the bottom of the board!!"
Changed lines of the file:
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@@
 have gnd/power and sometimes have
 power/gnd.  R30 &amp; R31 are 0 Ohm
-resistors on the top of the board let
-you select the screen type
+resistors on the top of the board that
+let you select the screen type
 When assembling make sure you put
 them in the right place or they will be
-hard to fix!!  If there is any doubt put
-them on the bottom of the board!!</text>
+hard to fix!! </text>
 <text x="269.24" y="10.16" size="1.778" layer="97">2.1</text>
 <text x="76.2" y="45.72" size="1.778" layer="97">J6</text>
@@
 <text x="27.94" y="66.04" size="1.778" layer="97">CY8C4247AZI-M485</text>
 <text x="121.92" y="5.08" size="3.81" layer="97">CY8CKIT-032</text>
+<text x="91.44" y="58.42" size="1.778" layer="97">P37 should be a direct path to thermistor
+ground</text>
 </plain>
 <instances>
@@
 <text x="170.18" y="5.08" size="5.08" layer="97">Sensors</text>
 <text x="104.14" y="93.98" size="1.778" layer="97" rot="R90">10K</text>
-<text x="134.62" y="71.12" size="1.778" layer="97" rot="R180">2.1</text>
 <text x="220.98" y="7.62" size="1.778" layer="97" rot="R180">2.1</text>
 <text x="180.34" y="25.4" size="3.81" layer="97">CY8CKIT-032</text>
