File: ww101-shield/eagle/ww101board.sch (EAGLE design)
At the start: 66 parts, among them J6 U8G-096-OLED, J7 0, U7 CY8C4A45-48

Commit message: a number of small changes to the 2.2 baord
Connections:
- net UARTRX: now also U7.P1[0]; no longer U7.P1[1]
- net UARTTX: now also U7.P1[1]; no longer U7.P1[0]
Other:
- note added: "U7"
Changed lines of the file:
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@@
 <text x="91.44" y="58.42" size="1.778" layer="97">P37 should be a direct path to thermistor
 ground</text>
+<text x="38.1" y="60.96" size="1.778" layer="97">U7</text>
 </plain>
 <instances>
@@
 <net name="UARTTX" class="0">
 <segment>
-<pinref part="U7" gate="G$1" pin="P1[0]"/>
-<wire x1="25.4" y1="88.9" x2="25.4" y2="99.06" width="0.1524" layer="91"/>
-<label x="25.4" y="91.44" size="1.778" layer="95" rot="R90"/>
+<pinref part="U7" gate="G$1" pin="P1[1]"/>
+<wire x1="7.62" y1="78.74" x2="-5.08" y2="78.74" width="0.1524" layer="91"/>
+<label x="-2.54" y="78.74" size="1.778" layer="95"/>
 </segment>
 </net>
@@
 <wire x1="53.34" y1="40.64" x2="53.34" y2="30.48" width="0.1524" layer="91"/>
 <label x="53.34" y="30.48" size="1.778" layer="95" rot="R90"/>
-</segment>
-</net>
-<net name="UARTRX" class="0">
-<segment>
-<pinref part="U7" gate="G$1" pin="P1[1]"/>
-<wire x1="7.62" y1="78.74" x2="-5.08" y2="78.74" width="0.1524" layer="91"/>
-<label x="-2.54" y="78.74" size="1.778" layer="95"/>
 </segment>
 </net>
@@
 </segment>
 </net>
+<net name="UARTRX" class="0">
+<segment>
+<pinref part="U7" gate="G$1" pin="P1[0]"/>
+<wire x1="25.4" y1="88.9" x2="25.4" y2="99.06" width="0.1524" layer="91"/>
+<label x="25.4" y="91.44" size="1.778" layer="95" rot="R90"/>
+</segment>
+</net>
