File: ww101-shield/eagle/ww101board.sch (EAGLE design)
At the start: 68 parts, among them J6 U8G-096-OLED, J7 0, U7 CY8C4A45-48

Commit message: Hopefully final V2.2 board
Connections:
- net GND: now also C15.1
- net VCC: no longer C15.1
Changed lines of the file:
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@@
 <part name="SUPPLY23" library="supply2" library_urn="urn:adsk.eagle:library:372" deviceset="GND" device=""/>
 <part name="SUPPLY33" library="supply2" library_urn="urn:adsk.eagle:library:372" deviceset="GND" device=""/>
+<part name="SUPPLY37" library="supply2" library_urn="urn:adsk.eagle:library:372" deviceset="GND" device=""/>
 </parts>
 <sheets>
@@
 <instance part="U$4" gate="G$1" x="73.66" y="0"/>
 <instance part="U$7" gate="G$1" x="111.76" y="167.64"/>
+<instance part="SUPPLY37" gate="GND" x="86.36" y="114.3" rot="R90"/>
 </instances>
 <busses>
@@
 <label x="76.2" y="55.88" size="1.778" layer="95"/>
 </segment>
+<segment>
+<pinref part="C15" gate="G$1" pin="1"/>
+<wire x1="78.74" y1="114.3" x2="83.82" y2="114.3" width="0.1524" layer="91"/>
+<pinref part="SUPPLY37" gate="GND" pin="GND"/>
+</segment>
 </net>
 <net name="CBLED2" class="0">
@@
 <segment>
 <pinref part="R22" gate="R" pin="1"/>
-<wire x1="78.74" y1="121.92" x2="83.82" y2="121.92" width="0.1524" layer="91"/>
 <pinref part="SUPPLY17" gate="G$1" pin="VCC"/>
-<pinref part="C15" gate="G$1" pin="1"/>
-<wire x1="83.82" y1="121.92" x2="91.44" y2="121.92" width="0.1524" layer="91"/>
-<wire x1="78.74" y1="114.3" x2="83.82" y2="114.3" width="0.1524" layer="91"/>
-<wire x1="83.82" y1="114.3" x2="83.82" y2="121.92" width="0.1524" layer="91"/>
-<junction x="83.82" y="121.92"/>
-</segment>
-</net>
+<wire x1="78.74" y1="121.92" x2="91.44" y2="121.92" width="0.1524" layer="91"/>
+</segment>
+</net>

Commit message: Version 2.2 of board files.
Parts:
- removed U$7: CYLOGO-SILK, ww101board:CYLOGO-SILK
- J5: value (none) -> vcc
- R32: value (none) -> 3.3v
Other:
- note added: "2.2"
- note added: "630-60500-01"
- note added: "CY8C4A45AZI-483"
- note added: "CY8CKIT-032 PSoC 4 AFE Shield"
- note added: "PSoC Analog Coprocessor"
- note added: "Power Selection Jumper"
- note added: "R18, R19, R20, R21 are 0 ohm resistors"
- note added: "Sensor Interface"
- note removed: "2.1"
- note removed: "CY8C4247AZI-M485"
- note removed: "CY8CKIT-032"
- note removed: "Flip RX/TX"
- note removed: "PSoC"
- note removed: "Power"
- note removed: "R26/R27 make this look like a "real" LED"
- note removed: "Sensors"
